Commit message: fix: change the dimension order to l,w,h instead of w,l,h

File: description/urdf/diffbot_description.urdf.xacro (robot description, xacro)
@@ -5,7 +5,7 @@
   <xacro:property name="PI" value="3.1415926535897931"/>
   <xacro:property name="base_mass" value="1" /> <!-- arbitrary value for base mass -->
+  <xacro:property name="base_length" value="0.2" />
   <xacro:property name="base_width" value="0.10" />
-  <xacro:property name="base_length" value="0.2" />
-  <xacro:property name="base_height" value="0.03" />
+  <xacro:property name="base_height" value="0.0447" />
   <xacro:property name="wheel_mass" value="0.2" /> <!-- arbitrary value for wheel mass -->
   <xacro:property name="wheel_len" value="0.029" />
@@ -19,5 +19,5 @@
       <origin xyz="0 0 0" rpy="0 0 0"/>
       <geometry>
-        <box size="${base_width} ${base_length} ${base_height}"/>
+        <box size="${base_length} ${base_width} ${base_height}"/>
       </geometry>
     </collision>
@@ -25,5 +25,5 @@
       <origin xyz="0 0 ${base_height/2}" rpy="0 0 0"/>
       <geometry>
-        <box size="${base_width} ${base_length} ${base_height}"/>
+        <box size="${base_length} ${base_width} ${base_height}"/>
       </geometry>
       <material name="orange"/>
@@ -33,7 +33,7 @@
       <mass value="${base_mass}"/>
       <inertia
-        ixx="${base_mass / 12.0 * (base_length*base_length + base_height*base_height)}" ixy="0.0" ixz="0.0"
-        iyy="${base_mass / 12.0 * (base_height*base_height + base_width*base_width)}" iyz="0.0"
-        izz="${base_mass / 12.0 * (base_width*base_width + base_length*base_length)}"/>
+        ixx="${base_mass / 12.0 * (base_width*base_width + base_height*base_height)}" ixy="0.0" ixz="0.0"
+        iyy="${base_mass / 12.0 * (base_height*base_height + base_length*base_length)}" iyz="0.0"
+        izz="${base_mass / 12.0 * (base_length*base_length + base_width*base_width)}"/>
       </inertial>
     </link>
@@ -103,5 +103,5 @@
       <parent link="${prefix}base_link"/>
       <child link="${prefix}caster_frontal_wheel"/>
-      <origin xyz="${base_width/2 - caster_wheel_radius} 0 ${z_offset}" rpy="0 0 0"/>
+      <origin xyz="${base_length/2 + wheel_radius - caster_wheel_radius} 0 ${z_offset}" rpy="0 0 0"/>
     </joint>
     <!-- caster frontal wheel Link -->

Commit message: fix: round wheel lenght to 0.3

File: description/urdf/diffbot_description.urdf.xacro (robot description, xacro)
@@ -9,5 +9,5 @@
   <xacro:property name="base_height" value="0.0447" />
   <xacro:property name="wheel_mass" value="0.2" /> <!-- arbitrary value for wheel mass -->
-  <xacro:property name="wheel_len" value="0.029" />
+  <xacro:property name="wheel_len" value="0.03" />
   <xacro:property name="wheel_radius" value="0.0325" />
   <xacro:property name="caster_wheel_mass" value="0.1" /> <!-- arbitrary value for caster wheel mass -->

Commit message: fix: remove rear caster wheel

File: description/urdf/diffbot_description.urdf.xacro (robot description, xacro)
@@ -129,33 +129,4 @@
         </inertial>
       </link>
-    <joint name="${prefix}caster_rear_wheel_joint" type="fixed">
-      <parent link="${prefix}base_link"/>
-      <child link="${prefix}caster_rear_wheel"/>
-      <origin xyz="${-base_width/2 + caster_wheel_radius} 0 ${z_offset}" rpy="0 0 0"/>
-    </joint>
-    <!-- caster rear wheel Link -->
-    <link name="${prefix}caster_rear_wheel">
-      <collision>
-        <origin xyz="0 0 0" rpy="0 0 0"/>
-        <geometry>
-          <sphere radius="${caster_wheel_radius}"/>
-        </geometry>
-      </collision>
-      <visual>
-        <origin xyz="0 0 0" rpy="0 0 0"/>
-        <geometry>
-          <sphere radius="${caster_wheel_radius}"/>
-        </geometry>
-        <material name="white"/>
-      </visual>
-      <inertial>
-        <origin xyz="0 0 0" rpy="0 0 0"/>
-        <mass value="${caster_wheel_mass}"/>
-        <inertia
-          ixx="${caster_wheel_mass * 0.4 * (caster_wheel_radius * caster_wheel_radius)}" ixy="0.0" ixz="0.0"
-          iyy="${caster_wheel_mass * 0.4 * (caster_wheel_radius * caster_wheel_radius)}" iyz="0.0"
-          izz="${caster_wheel_mass * 0.4 * (caster_wheel_radius * caster_wheel_radius)}"/>
-        </inertial>
-      </link>
   </xacro:macro>
 </robot>

Commit message: fix: correct the base_link coordinates

File: description/urdf/diffbot_description.urdf.xacro (robot description, xacro)
@@ -17,5 +17,5 @@
   <link name="${prefix}base_link">
     <collision>
-      <origin xyz="0 0 0" rpy="0 0 0"/>
+      <origin xyz="${wheel_radius} 0 ${base_height/2}" rpy="0 0 0"/>
       <geometry>
         <box size="${base_length} ${base_width} ${base_height}"/>
@@ -23,5 +23,5 @@
     </collision>
     <visual>
-      <origin xyz="0 0 ${base_height/2}" rpy="0 0 0"/>
+      <origin xyz="${wheel_radius} 0 ${base_height/2}" rpy="0 0 0"/>
       <geometry>
         <box size="${base_length} ${base_width} ${base_height}"/>

Commit message: fix: correct the left and right wheel joint coordinates

File: description/urdf/diffbot_description.urdf.xacro (robot description, xacro)
@@ -41,5 +41,5 @@
       <parent link="${prefix}base_link"/>
       <child link="${prefix}left_wheel"/>
-      <origin xyz="0 -${base_width/2} ${z_offset}" rpy="0 0 0"/>
+      <origin xyz="0 -${base_width/2 + wheel_len/2.0} ${z_offset}" rpy="0 0 0"/>
       <axis xyz="0 1 0"/>
       <dynamics damping="0.2"/>
@@ -72,5 +72,5 @@
       <parent link="${prefix}base_link"/>
       <child link="${prefix}right_wheel"/>
-      <origin xyz="0 ${base_width/2} ${z_offset}" rpy="0 0 0"/>
+      <origin xyz="0 ${base_width/2 + wheel_len/2.0} ${z_offset}" rpy="0 0 0"/>
       <axis xyz="0 1 0"/>
       <dynamics damping="0.2"/>

Commit message: fix: add gazebo related libraries and plugins for simulation

File: description/urdf/diffbot_description.urdf.xacro (robot description, xacro)
@@ -1,4 +1,5 @@
 <?xml version="1.0"?>
 <robot xmlns:xacro="http://www.ros.org/wiki/xacro">
+  <!-- Diffbot Macro -->
   <xacro:macro name="diffbot" params="prefix">
   <!-- Constants for robot dimensions -->
@@ -36,97 +37,126 @@
         iyy="${base_mass / 12.0 * (base_height*base_height + base_length*base_length)}" iyz="0.0"
         izz="${base_mass / 12.0 * (base_length*base_length + base_width*base_width)}"/>
-      </inertial>
-    </link>
-    <joint name="${prefix}left_wheel_joint" type="continuous">
-      <parent link="${prefix}base_link"/>
-      <child link="${prefix}left_wheel"/>
-      <origin xyz="0 -${base_width/2 + wheel_len/2.0} ${z_offset}" rpy="0 0 0"/>
-      <axis xyz="0 1 0"/>
-      <dynamics damping="0.2"/>
-    </joint>
-    <!-- left wheel Link -->
-    <link name="${prefix}left_wheel">
-      <collision>
-        <origin xyz="0 0 0" rpy="${PI/2} 0 0"/>
-        <geometry>
-          <cylinder length="${wheel_len}" radius="${wheel_radius}"/>
-        </geometry>
-      </collision>
-      <visual>
-        <origin xyz="0 0 0" rpy="${PI/2} 0 0"/>
-        <geometry>
-          <cylinder length="${wheel_len}" radius="${wheel_radius}"/>
-        </geometry>
-        <material name="black"/>
-      </visual>
-      <inertial>
-        <origin xyz="0 0 0" rpy="${PI/2} 0 0"/>
-        <mass value="${wheel_mass}"/>
-        <inertia
-          ixx="${wheel_mass / 12.0 * (3*wheel_radius*wheel_radius + wheel_len*wheel_len)}" ixy="0.0" ixz="0.0"
-          iyy="${wheel_mass / 2.0 * wheel_radius*wheel_radius}" iyz="0.0"
-          izz="${wheel_mass / 12.0 * (3*wheel_radius*wheel_radius + wheel_len*wheel_len)}"/>
-        </inertial>
-      </link>
-    <joint name="${prefix}right_wheel_joint" type="continuous">
-      <parent link="${prefix}base_link"/>
-      <child link="${prefix}right_wheel"/>
-      <origin xyz="0 ${base_width/2 + wheel_len/2.0} ${z_offset}" rpy="0 0 0"/>
-      <axis xyz="0 1 0"/>
-      <dynamics damping="0.2"/>
-    </joint>
-    <!-- right wheel Link -->
-    <link name="${prefix}right_wheel">
-      <collision>
-        <origin xyz="0 0 0" rpy="${PI/2} 0 0"/>
-        <geometry>
-          <cylinder length="${wheel_len}" radius="${wheel_radius}"/>
-        </geometry>
-      </collision>
-      <visual>
-        <origin xyz="0 0 0" rpy="${PI/2} 0 0"/>
-        <geometry>
-          <cylinder length="${wheel_len}" radius="${wheel_radius}"/>
-        </geometry>
-        <material name="black"/>
-      </visual>
-      <inertial>
-        <origin xyz="0 0 0" rpy="${PI/2} 0 0"/>
-        <mass value="${wheel_mass}"/>
-        <inertia
-          ixx="${wheel_mass / 12.0 * (3*wheel_radius*wheel_radius + wheel_len*wheel_len)}" ixy="0.0" ixz="0.0"
-          iyy="${wheel_mass / 2.0 * wheel_radius*wheel_radius}" iyz="0.0"
-          izz="${wheel_mass / 12.0 * (3*wheel_radius*wheel_radius + wheel_len*wheel_len)}"/>
-        </inertial>
-      </link>
-    <joint name="${prefix}caster_frontal_wheel_joint" type="fixed">
-      <parent link="${prefix}base_link"/>
-      <child link="${prefix}caster_frontal_wheel"/>
-      <origin xyz="${base_length/2 + wheel_radius - caster_wheel_radius} 0 ${z_offset}" rpy="0 0 0"/>
-    </joint>
-    <!-- caster frontal wheel Link -->
-    <link name="${prefix}caster_frontal_wheel">
-      <collision>
-        <origin xyz="0 0 0" rpy="0 0 0"/>
-        <geometry>
-          <sphere radius="${caster_wheel_radius}"/>
-        </geometry>
-      </collision>
-      <visual>
-        <origin xyz="0 0 0" rpy="0 0 0"/>
-        <geometry>
-          <sphere radius="${caster_wheel_radius}"/>
-        </geometry>
-        <material name="white"/>
-      </visual>
-      <inertial>
-        <origin xyz="0 0 0" rpy="0 0 0"/>
-        <mass value="${caster_wheel_mass}"/>
-        <inertia
-          ixx="${caster_wheel_mass * 0.4 * (caster_wheel_radius * caster_wheel_radius)}" ixy="0.0" ixz="0.0"
-          iyy="${caster_wheel_mass * 0.4 * (caster_wheel_radius * caster_wheel_radius)}" iyz="0.0"
-          izz="${caster_wheel_mass * 0.4 * (caster_wheel_radius * caster_wheel_radius)}"/>
-        </inertial>
-      </link>
+    </inertial>
+  </link>
+  <!-- Left Wheel Joint -->
+  <joint name="${prefix}left_wheel_joint" type="continuous">
+    <parent link="${prefix}base_link"/>
+    <child link="${prefix}left_wheel"/>
+    <origin xyz="0 -${base_width/2 + wheel_len/2.0} ${z_offset}" rpy="0 0 0"/>
+    <axis xyz="0 1 0"/>
+    <dynamics damping="0.2"/>
+  </joint>
+  <!-- left wheel Link -->
+  <link name="${prefix}left_wheel">
+    <collision>
+      <origin xyz="0 0 0" rpy="${PI/2} 0 0"/>
+      <geometry>
+        <cylinder length="${wheel_len}" radius="${wheel_radius}"/>
+      </geometry>
+    </collision>
+    <visual>
+      <origin xyz="0 0 0" rpy="${PI/2} 0 0"/>
+      <geometry>
+        <cylinder length="${wheel_len}" radius="${wheel_radius}"/>
+      </geometry>
+      <material name="black"/>
+    </visual>
+    <inertial>
+      <origin xyz="0 0 0" rpy="${PI/2} 0 0"/>
+      <mass value="${wheel_mass}"/>
+      <inertia
+        ixx="${wheel_mass / 12.0 * (3*wheel_radius*wheel_radius + wheel_len*wheel_len)}" ixy="0.0" ixz="0.0"
+        iyy="${wheel_mass / 2.0 * wheel_radius*wheel_radius}" iyz="0.0"
+        izz="${wheel_mass / 12.0 * (3*wheel_radius*wheel_radius + wheel_len*wheel_len)}"/>
+    </inertial>
+  </link>
+  <!-- Right Wheel Joint -->
+  <joint name="${prefix}right_wheel_joint" type="continuous">
+    <parent link="${prefix}base_link"/>
+    <child link="${prefix}right_wheel"/>
+    <origin xyz="0 ${base_width/2 + wheel_len/2.0} ${z_offset}" rpy="0 0 0"/>
+    <axis xyz="0 1 0"/>
+    <dynamics damping="0.2"/>
+  </joint>
+  <!-- right wheel Link -->
+  <link name="${prefix}right_wheel">
+    <collision>
+      <origin xyz="0 0 0" rpy="${PI/2} 0 0"/>
+      <geometry>
+        <cylinder length="${wheel_len}" radius="${wheel_radius}"/>
+      </geometry>
+    </collision>
+    <visual>
+      <origin xyz="0 0 0" rpy="${PI/2} 0 0"/>
+      <geometry>
+        <cylinder length="${wheel_len}" radius="${wheel_radius}"/>
+      </geometry>
+      <material name="black"/>
+    </visual>
+    <inertial>
+      <origin xyz="0 0 0" rpy="${PI/2} 0 0"/>
+      <mass value="${wheel_mass}"/>
+      <inertia
+        ixx="${wheel_mass / 12.0 * (3*wheel_radius*wheel_radius + wheel_len*wheel_len)}" ixy="0.0" ixz="0.0"
+        iyy="${wheel_mass / 2.0 * wheel_radius*wheel_radius}" iyz="0.0"
+        izz="${wheel_mass / 12.0 * (3*wheel_radius*wheel_radius + wheel_len*wheel_len)}"/>
+    </inertial>
+  </link>
+  <!-- Caster Frontal Wheel Joint -->
+  <joint name="${prefix}caster_frontal_wheel_joint" type="fixed">
+    <parent link="${prefix}base_link"/>
+    <child link="${prefix}caster_frontal_wheel"/>
+    <origin xyz="${base_length/2 + wheel_radius - caster_wheel_radius} 0 ${z_offset}" rpy="0 0 0"/>
+  </joint>
+  <!-- caster frontal wheel Link -->
+  <link name="${prefix}caster_frontal_wheel">
+    <collision>
+      <origin xyz="0 0 0" rpy="0 0 0"/>
+      <geometry>
+        <sphere radius="${caster_wheel_radius}"/>
+      </geometry>
+    </collision>
+    <visual>
+      <origin xyz="0 0 0" rpy="0 0 0"/>
+      <geometry>
+        <sphere radius="${caster_wheel_radius}"/>
+      </geometry>
+      <material name="white"/>
+    </visual>
+    <inertial>
+      <origin xyz="0 0 0" rpy="0 0 0"/>
+      <mass value="${caster_wheel_mass}"/>
+      <inertia
+        ixx="${caster_wheel_mass * 0.4 * (caster_wheel_radius * caster_wheel_radius)}" ixy="0.0" ixz="0.0"
+        iyy="${caster_wheel_mass * 0.4 * (caster_wheel_radius * caster_wheel_radius)}" iyz="0.0"
+        izz="${caster_wheel_mass * 0.4 * (caster_wheel_radius * caster_wheel_radius)}"/>
+    </inertial>
+  </link>
+  <!-- Laser Joint -->
+  <joint name="${prefix}laser_joint" type="fixed">
+    <parent link="${prefix}base_link"/>
+    <child link="${prefix}laser_frame"/>
+    <origin xyz="0.1 0 0.08" rpy="0 0 0"/>
+  </joint>
+  <link name="${prefix}laser_frame">
+    <visual>
+      <geometry>
+        <cylinder radius="0.05" length="0.04"/>
+      </geometry>
+      <material name="black"/>
+    </visual>
+    <collision>
+      <geometry>
+        <cylinder radius="0.05" length="0.04"/>
+      </geometry>
+    </collision>
+    <inertial>
+      <mass value="0.1"/>
+      <inertia
+        ixx="0.000041" ixy="0.0" ixz="0.0"
+        iyy="0.000041" iyz="0.0"
+        izz="0.000125"/>
+    </inertial>
+  </link>
   </xacro:macro>
 </robot>

Commit message: fix: adjust dimensions for resembalnce with real bot

File: description/urdf/diffbot_description.urdf.xacro (robot description, xacro)
@@ -13,5 +13,5 @@
   <xacro:property name="wheel_radius" value="0.0325" />
   <xacro:property name="caster_wheel_mass" value="0.1" /> <!-- arbitrary value for caster wheel mass -->
-  <xacro:property name="caster_wheel_radius" value="0.01625" />
+  <xacro:property name="caster_wheel_radius" value="0.0325" />
   <xacro:property name="z_offset" value="-${base_height/2}" /> <!-- Space btw top of beam and the each joint -->
   <!-- Base Link -->
@@ -137,5 +137,5 @@
     <parent link="${prefix}base_link"/>
     <child link="${prefix}laser_frame"/>
-    <origin xyz="0.1 0 0.08" rpy="0 0 0"/>
+    <origin xyz="0.1 0 ${base_height + 0.02}" rpy="0 0 0"/>
   </joint>
   <link name="${prefix}laser_frame">

Commit message: test: test by changing axis of wheels for stability

File: description/urdf/diffbot_description.urdf.xacro (robot description, xacro)
@@ -63,5 +63,5 @@
     </visual>
     <inertial>
-      <origin xyz="0 0 0" rpy="${PI/2} 0 0"/>
+      <origin xyz="0 0 0" rpy="0 0 0"/>
       <mass value="${wheel_mass}"/>
       <inertia
@@ -95,5 +95,5 @@
     </visual>
     <inertial>
-      <origin xyz="0 0 0" rpy="${PI/2} 0 0"/>
+      <origin xyz="0 0 0" rpy="0 0 0"/>
       <mass value="${wheel_mass}"/>
       <inertia

Commit message: fix: fix caster wheel joint coordinates

File: description/urdf/diffbot_description.urdf.xacro (robot description, xacro)
@@ -18,5 +18,5 @@
   <link name="${prefix}base_link">
     <collision>
-      <origin xyz="${wheel_radius} 0 ${base_height/2}" rpy="0 0 0"/>
+      <origin xyz="0 0 ${base_height/2}" rpy="0 0 0"/>
       <geometry>
         <box size="${base_length} ${base_width} ${base_height}"/>
@@ -24,5 +24,5 @@
     </collision>
     <visual>
-      <origin xyz="${wheel_radius} 0 ${base_height/2}" rpy="0 0 0"/>
+      <origin xyz="0 0 ${base_height/2}" rpy="0 0 0"/>
       <geometry>
         <box size="${base_length} ${base_width} ${base_height}"/>
@@ -31,5 +31,5 @@
     </visual>
     <inertial>
-      <origin xyz="0 0 0" rpy="0 0 0"/>
+      <origin xyz="0 0 ${base_height/2}" rpy="0 0 0"/>
       <mass value="${base_mass}"/>
       <inertia
@@ -107,5 +107,5 @@
     <parent link="${prefix}base_link"/>
     <child link="${prefix}caster_frontal_wheel"/>
-    <origin xyz="${base_length/2 + wheel_radius - caster_wheel_radius} 0 ${z_offset}" rpy="0 0 0"/>
+    <origin xyz="${base_length/2} 0 ${z_offset}" rpy="0 0 0"/>
   </joint>
   <!-- caster frontal wheel Link -->
